Commit message: Added some fixes
Signed-off-by: ahcorde <ahcorde@gmail.com>

File: ignition_ros2_control_demos/urdf/test_cart_velocity.xacro.urdf (robot description, URDF)
Before this commit: robot cartopole, 3 links, 2 joints
Links:
- removed link world
- added link imu, mass 0.1
- added link leg1, mass 1; collision cylinder length=1.0 radius=0.2; visual cylinder length=1.0 radius=0.2
- added link leg2, mass 1; collision cylinder length=1.0 radius=0.2; visual cylinder length=1.0 radius=0.2
Joints:
- removed joint world_to_base
- added joint cart_to_imu: type fixed, parent cart, child imu, origin xyz=0.0 0.0 0.0
- added joint slider_to_leg1: type fixed, parent slideBar, child leg1, origin xyz=-15.0 0.0 0.5
- added joint slider_to_leg2: type fixed, parent slideBar, child leg2, origin xyz=15 0.0 0.5
