Commit message: Improved inertial gripper
Signed-off-by: ahcorde <ahcorde@gmail.com>

File: gz_ros2_control_demos/urdf/test_gripper_mimic_joint.xacro.urdf (robot description, URDF)
Before this commit: robot gripper, 4 links, 3 joints
Links:
- link finger_left: mass 5 -> 4
- link finger_right: mass 5 -> 4

Commit message: Fixed gripper xacro
Signed-off-by: ahcorde <ahcorde@gmail.com>

File: gz_ros2_control_demos/urdf/test_gripper_mimic_joint.xacro.urdf (robot description, URDF)
Before this commit: robot gripper, 4 links, 3 joints
Joints:
- joint left_finger_joint: limit lower=0 upper=0.38 effort=1000.0 velocity=10 -> lower=-0.05 upper=0.39 effort=100000.0 velocity=1
- joint right_finger_joint: limit lower=0 upper=0.38 effort=1000.0 velocity=10 -> lower=-0.05 upper=0.39 effort=100000.0 velocity=1
