Commit message: Added some fixes
Signed-off-by: ahcorde <ahcorde@gmail.com>

File: gz_ros2_control_demos/urdf/test_cart_position.xacro.urdf (robot description, URDF)
Before this commit: robot cartopole, 3 links, 2 joints
Links:
- link cart: geometry collision box size=0.5 0.5 0.2; visual box size=0.5 0.5 0.2
- link slideBar: geometry collision box size=30 0.05 0.05; visual box size=30 0.05 0.05

File: gz_ros2_control_demos/urdf/test_cart_velocity.xacro.urdf (robot description, URDF)
Before this commit: robot cartopole, 5 links, 4 joints
Links:
- added link world
Joints:
- added joint world_to_base: type fixed, parent world, child slideBar, origin xyz=0 0 1 rpy=0 0 0

File: gz_ros2_control_demos/urdf/test_gripper_mimic_joint.xacro.urdf (robot description, URDF)
Before this commit: robot gripper, 4 links, 3 joints
Links:
- link base: geometry collision box size=0.5 1 1; visual box size=0.5 1 1
Joints:
- joint left_finger_joint: limit lower=-0.05 upper=0.39 effort=100000.0 velocity=1 -> lower=0 upper=0.38 effort=1000.0 velocity=10
- joint right_finger_joint: limit lower=-0.05 upper=0.39 effort=100000.0 velocity=1 -> lower=0 upper=0.38 effort=1000.0 velocity=10

Commit message: Renamed ign to gz (#67)
Signed-off-by: Alejandro Hernández Cordero <ahcorde@gmail.com>

File: gz_ros2_control_demos/urdf/test_cart_position.xacro.urdf (robot description, URDF)
Before this commit: robot cartopole, 3 links, 2 joints
Links:
- link cart: geometry collision box size=0.5 0.5 0.2; visual box size=0.5 0.5 0.2
- link slideBar: geometry collision box size=30 0.05 0.05; visual box size=30 0.05 0.05
