Commit message: Change initial pose of pendulum

File: gz_ros2_control_demos/urdf/test_pendulum_effort.xacro.urdf (robot description, URDF)
Before this commit: robot pendulum on cart, 2 links, 3 joints
Joints:
- joint cart_to_pendulum: origin xyz=0.0 0.35 0.0 rpy=0 0.1 0 -> xyz=0.0 0.35 0.0 rpy=0 ${pi} 0
