Commit message: Make position and effort version of pendulum equal

File: gz_ros2_control_demos/urdf/test_pendulum_position.xacro.urdf (robot description, URDF)
Before this commit: robot cartopole, 4 links, 3 joints
Links:
- removed link cart
- removed link pendulum
Joints:
- joint cart_to_pendulum: limit lower=-10000 upper=10000 effort=1000.0 velocity=30 -> lower=-100000 upper=100000 effort=10000.0 velocity=100000; origin xyz=0.0 0.35 0.0 -> xyz=0.0 0.35 0.0 rpy=0 ${pi} 0
