Commit message: added steer inertial tag

File: gz_ros2_control_demos/urdf/test_ackermann_drive.xacro.urdf (robot description, URDF)
Before this commit: robot tricycle_drive, 8 links, 7 joints
Links:
- link left_wheel_steering: mass None -> 0.1
- link right_wheel_steering: mass None -> 0.1

Commit message: updated documentation

File: gz_ros2_control_demos/urdf/test_ackermann_drive.xacro.urdf (robot description, URDF)
Before this commit: robot tricycle_drive, 8 links, 7 joints
Joints:
- joint front_left_wheel_joint: mimic joint=rear_left_wheel_joint -> (none)
- joint front_right_wheel_joint: mimic joint=rear_right_wheel_joint -> (none)
