Commit message: Restore Humble's upstream gz_system.cpp and index.rst, and update gripper YAML/URDF files to match Jazzy versions

File: gz_ros2_control_demos/urdf/test_gripper_mimic_joint_position.xacro.urdf (robot description, URDF)
Before this commit: robot gripper, 4 links, 3 joints
Links:
- link base: geometry collision box size=0.5 1 1; visual box size=0.5 1 1
- link finger_left: mass 5 -> 4
- link finger_right: mass 5 -> 4
