Commit message: Apply the mimic joint offset in GazeboSimSystem::write
URDF defines a mimic joint as follower = multiplier * driver + offset.
MimicJoint::offset reaches the plugin and is printed at startup, but the
arithmetic that drives the follower never referenced it, so a URDF
declaring an offset produced a follower tracking multiplier * driver with
the offset silently dropped.

gazebo_ros2_control, the sibling plugin, already applies the full form in
gazebo_system.cpp.

The existing mimic fixtures declare <mimic joint="..."/> with no offset,
so the default of zero made this invisible to the test suite. The position
gripper fixture now declares an explicit multiplier and offset, and the
test asserts the follower satisfies the URDF relationship once it settles.

Verified in Gazebo 8.11 on a gripper with offset 0.05: before the change
the follower held 0.1500 against an expected 0.2000, an error equal to the
dropped offset; after it, the error is zero.

Reported with analysis and a patch by @omnilink-tech in #952.

Signed-off-by: Puja Chaudhury <61319491+catplotlib@users.noreply.github.com>

File: gz_ros2_control_demos/urdf/test_gripper_mimic_joint_position.xacro.urdf (robot description, URDF)
Before this commit: robot gripper, 4 links, 3 joints
Joints:
- joint left_finger_joint: mimic joint=right_finger_joint -> joint=right_finger_joint multiplier=1.0 offset=0.05
