Commit message: Update limits

File: gz_ros2_control_demos/urdf/test_tricycle_drive.xacro.urdf (robot description, URDF)
Before this commit: robot tricycle_drive, 6 links, 5 joints
Joints:
- joint steering_joint: limit (none) -> lower=-1.57 upper=1.57 effort=100 velocity=1
- joint traction_joint: limit (none) -> effort=100 velocity=1
