Commit message: Feedback and fix
Signed-off-by: ahcorde <ahcorde@gmail.com>

File: ign_ros2_control_demos/urdf/test_diff_drive.xacro.urdf (robot description, URDF)
Before this commit: robot diff_drive, 4 links, 3 joints
Links:
- link caster: mass 1 -> 0.005

Commit message: Adapt pid params for examples.

File: ign_ros2_control_demos/urdf/test_diff_drive.xacro.urdf (robot description, URDF)
Before this commit: robot diff_drive, 4 links, 3 joints
Joints:
- joint left_wheel_joint: limit (none) -> effort=1000.0 velocity=30
- joint right_wheel_joint: limit (none) -> effort=1000.0 velocity=30

File: ign_ros2_control_demos/urdf/test_tricycle_drive.xacro.urdf (robot description, URDF)
Before this commit: robot tricycle_drive, 6 links, 5 joints
Joints:
- joint left_wheel_joint: limit (none) -> effort=1000.0 velocity=30
- joint right_wheel_joint: limit (none) -> effort=1000.0 velocity=30
- joint steering_joint: limit (none) -> effort=1000.0 velocity=30
- joint traction_joint: limit (none) -> effort=1000.0 velocity=30
